File: DA SBROGLIARE/lickshot_delay.kicad_sch (KiCad schematic)
At the start: 75 parts, among them Q1 2N3904, SW1 SW_DPDT_x2, SW2 SW_DPDT_x2, U1 4069, U2 4046, U3 TL072, U4 L7805, U5 PT2399

Commit message: Ordinati tutti i componenti, mancano da fare le tracce
Parts:
- added J1: Conn_01x02, Connector_Wire:SolderWire-0.5sqmm_1x02_P4.6mm_D0.9mm_OD2.1mm, symbol Connector_Generic:Conn_01x02
- added J2: 9v, Connector_Wire:SolderWire-0.5sqmm_1x02_P4.6mm_D0.9mm_OD2.1mm, symbol Connector_Generic:Conn_01x02
- added SW3: SW_SPST, Connector_Wire:SolderWire-0.5sqmm_1x02_P4.6mm_D0.9mm_OD2.1mm, symbol Switch:SW_SPST
- C10: value 47nf -> 4.7n
- C16: footprint Monkey_Riot_Pedals_Library:CP_Electro_D6.3mm_P2.50mm -> Monkey_Riot_Pedals_Library:CP_Electro_Radial_D5.0mm_P2.50mm
- D4: footprint Diode_THT:D_DO-41_SOD81_P10.16mm_Horizontal -> Monkey_Riot_Pedals_Library:DIODE_DO-35_SOD27_P7.62mm_Horizontal
Connections:
- net GND: now also J1.2 (Pin_2), J2.1 (Pin_1)
- net at C5.1, R14.2: now also SW3.2 (B); no longer R8.1, R9.2
- net at R10.1: now also J1.1 (Pin_1)
- net +9V: no longer names the net of D4.2 (A)
- net +9V: now also J2.2 (Pin_2)
- new net: R8.1, R9.2, SW3.1 (A)
- no-connect marks 1 -> 0
